Commit message: added xacro files

File: description/ros2_control/keya.ros2_control.xacro (robot description, xacro)
@@ -4,8 +4,9 @@
         <ros2_control name="{name}" type="actuator">
             <hardware>
+                <plugin>keya_driver_hardware_interface/KeyaDriverHW</plugin>
                 <param name="device_id">can0</param>
                 <param name="can_id_list">{1}</param>
             </hardware>
-            <joint name="${prefix}steering_motor">
+            <joint name="${prefix}_steering_motor">
                 <command_interface name="position"/>
                 <state_interface name="position"/>

Commit message: edited xacro files

File: description/ros2_control/keya.ros2_control.xacro (robot description, xacro)
@@ -2,14 +2,13 @@
 <robot xmlns:xacro="http://www.ros.org/wiki/xacro">
     <xacro:macro name="keya_ros2_control" params="name prefix">
-        <ros2_control name="{name}" type="actuator">
+        <ros2_control name="${name}" type="actuator">
             <hardware>
                 <plugin>keya_driver_hardware_interface/KeyaDriverHW</plugin>
-                <param name="device_id">can0</param>
-                <param name="can_id_list">{1}</param>
+                <!-- <param name="device_id">can0</param> -->
+                <!-- <param name="can_id_list">{1}</param> -->
             </hardware>
             <joint name="${prefix}_steering_motor">
                 <command_interface name="position"/>
                 <state_interface name="position"/>
-                <state_interface name="velocity"/>
             </joint>
         </ros2_control>

File: description/ros2_control/keya.urdf.xacro (robot description, xacro)
@@ -6,6 +6,6 @@
     <xacro:property name="wheel_radius" value="0.04" />
     <xacro:property name="wheel_height" value="0.095" />
-    <xacro:macro name="Keya" params="parent prefix">
-        <link name="{prefix}_base_link">
+    <xacro:macro name="keya" params="parent prefix">
+        <link name="${prefix}_base_link">
             <visual>
                 <geometry>
@@ -40,4 +40,5 @@
             <origin xyz="0 0 0" rpy="0 0 0" />
             <axis xyz="0 0 1" />
+            <limit lower="0" upper="3.14" velocity="0.5" effort="1.0" />
         </joint>
     </xacro:macro>

File: description/ros2_control/keya_world.xacro (robot description, xacro)
@@ -1,9 +1,9 @@
 <?xml version="1.0"?>
-<!-- Revolute-Revolute Manipulator -->
+<!-- KEYA Automatic Steering Motor -->
 <robot xmlns:xacro="http://www.ros.org/wiki/xacro" name="keya_world">
-  <!-- Import RRBot URDF -->
-  <xacro:include filename="$(find ros2_keya_driver)/description/keya.urdf.xacro" />
-  <!-- Import RRBot ros2_control description -->
-  <xacro:include filename="$(find ros2_keya_driver)/description/keya.ros2_control.xacro" />
+  <!-- Import Keya URDF -->
+  <xacro:include filename="$(find ros2_keya_driver)/description/ros2_control/keya.urdf.xacro" />
+  <!-- Import Keya ros2_control description -->
+  <xacro:include filename="$(find ros2_keya_driver)/description/ros2_control/keya.ros2_control.xacro" />
   <xacro:arg name="prefix" default="motor" />
   <xacro:arg name="parent" default="world" />

Commit message: debugged read()

File: description/ros2_control/keya.ros2_control.xacro (robot description, xacro)
@@ -8,7 +8,7 @@
                 <!-- <param name="can_id_list">{1}</param> -->
             </hardware>
-            <joint name="${prefix}_steering_motor">
-                <command_interface name="position"/>
-                <state_interface name="position"/>
+            <joint name="${prefix}_joint">
+                <command_interface name="position" />
+                <state_interface name="position" />
             </joint>
         </ros2_control>

File: description/ros2_control/keya.urdf.xacro (robot description, xacro)
@@ -23,5 +23,5 @@
             <origin xyz="0 0 0" rpy="0 0 0" />
         </joint>
-        <link name="${prefix}_wheel">
+        <link name="${prefix}_wheel_link">
             <visual>
                 <geometry>
@@ -37,5 +37,5 @@
         <joint name="${prefix}_joint" type="revolute">
             <parent link="${prefix}_base_link" />
-            <child link="${prefix}_wheel" />
+            <child link="${prefix}_wheel_link" />
             <origin xyz="0 0 0" rpy="0 0 0" />
             <axis xyz="0 0 1" />
