Commit message: added transmission_interface

File: description/keya.ros2_control.xacro (robot description, xacro)
@@ -12,4 +12,10 @@
                 <state_interface name="position" />
             </joint>
+            <transmission name="${prefix}_transmission">
+                <plugin>transmission_interface/SimpleTransmission</plugin>
+                <joint name="${prefix}_joint" role="${prefix}_joint">
+                    <mechanical_reduction>22.44</mechanical_reduction>
+                </joint>
+            </transmission>
         </ros2_control>
     </xacro:macro>

Commit message: fix min max

File: description/keya.ros2_control.xacro (robot description, xacro)
@@ -10,6 +10,6 @@
             <joint name="${prefix}_joint">
                 <command_interface name="position" >
-                    <param name="min">-0.26</param>
-                    <param name="max">0.26</param>
+                    <param name="min">-0.5</param>
+                    <param name="max">0.5</param>
                 </command_interface>
                 <state_interface name="position" />

File: description/keya.urdf.xacro (robot description, xacro)
@@ -40,5 +40,5 @@
             <origin xyz="0 0 0" rpy="0 0 0" />
             <axis xyz="0 0 1" />
-            <limit lower="0" upper="3.14" velocity="0.5" effort="1.0" />
+            <limit lower="-0.5" upper="0.5" velocity="0.5" effort="1.0" />
         </joint>
     </xacro:macro>
